File: Schematics/MirrorController.brd (EAGLE design)
At the start: 100 x 80 mm, 23 parts, among them T1 2N2222, U1 ATMEGA328P_PDIP

Commit message: +I2C Support and temp files removed
Parts:
- removed S1, S2, S3, S4, S5, S6, S7: SWITCH-MOMENTARY-2PTH, SparkFun-Electromechanical:TACTILE-PTH
- R2, R8: value (none) -> 3.9K
- R3, R9: value (none) -> 1K
- R4, R7: value (none) -> 27K
- R5: value (none) -> 10K
Connections:
- net GND: no longer S1.3, S2.3, S3.3, S4.3, S5.3, S6.3, S7.3
- net GPIO21: now also U1.25; no longer U1.28
- net N$1: no longer S1.1
- net N$2: no longer S2.1
- net N$3: no longer S3.1
- net N$4: no longer S4.1
- net N$5: no longer S5.1
- net N$6: no longer S6.1
- net N$7: no longer S7.1
Changed lines of the file:
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@@
 <elements>
 <element name="R1" library="SparkFun-Resistors" package="AXIAL-0.4" value="10K" x="-19.05" y="13.97"/>
-<element name="R2" library="SparkFun-Resistors" package="AXIAL-0.4" value="" x="-31.75" y="13.97"/>
-<element name="R3" library="SparkFun-Resistors" package="AXIAL-0.4" value="" x="-19.05" y="19.05"/>
-<element name="R4" library="SparkFun-Resistors" package="AXIAL-0.4" value="" x="-31.75" y="19.05"/>
-<element name="R5" library="SparkFun-Resistors" package="AXIAL-0.4" value="" x="-19.05" y="24.13"/>
+<element name="R2" library="SparkFun-Resistors" package="AXIAL-0.4" value="3.9K" x="-31.75" y="13.97"/>
+<element name="R3" library="SparkFun-Resistors" package="AXIAL-0.4" value="1K" x="-19.05" y="19.05"/>
+<element name="R4" library="SparkFun-Resistors" package="AXIAL-0.4" value="27K" x="-31.75" y="19.05"/>
+<element name="R5" library="SparkFun-Resistors" package="AXIAL-0.4" value="10K" x="-19.05" y="24.13"/>
 <element name="R6" library="SparkFun-Resistors" package="AXIAL-0.4" value="10K" x="-31.75" y="24.13"/>
-<element name="R7" library="SparkFun-Resistors" package="AXIAL-0.4" value="" x="-19.05" y="29.21"/>
-<element name="R8" library="SparkFun-Resistors" package="AXIAL-0.4" value="" x="-31.75" y="29.21"/>
-<element name="R9" library="SparkFun-Resistors" package="AXIAL-0.4" value="" x="-19.05" y="34.29"/>
+<element name="R7" library="SparkFun-Resistors" package="AXIAL-0.4" value="27K" x="-19.05" y="29.21"/>
+<element name="R8" library="SparkFun-Resistors" package="AXIAL-0.4" value="3.9K" x="-31.75" y="29.21"/>
+<element name="R9" library="SparkFun-Resistors" package="AXIAL-0.4" value="1K" x="-19.05" y="34.29"/>
 <element name="U1" library="SparkFun-DigitalIC" package="DIL28-3" value="ATMEGA328P_PDIP" x="-31.75" y="6.35"/>
 <element name="T1" library="adafruit" package="TO92-EBC-OVAL" value="2N2222" x="-54.61" y="5.08"/>
@@
 <element name="D1" library="SparkFun-LED" package="LED5MM" value="BLUE" x="-54.61" y="-13.97"/>
 <element name="R12" library="SparkFun-Resistors" package="AXIAL-0.4" value="220" x="-50.8" y="-20.32"/>
-<element name="S1" library="SparkFun-Electromechanical" package="TACTILE-PTH" value="SWITCH-MOMENTARY-2PTH" x="-63.5" y="-17.78">
-<attribute name="PROD_ID" value=" SWCH-08441" x="-63.5" y="-17.78" size="1.778" layer="27" display="off"/>
-</element>
-<element name="S2" library="SparkFun-Electromechanical" package="TACTILE-PTH" value="SWITCH-MOMENTARY-2PTH" x="-72.39" y="-17.78">
-<attribute name="PROD_ID" value=" SWCH-08441" x="-72.39" y="-17.78" size="1.778" layer="27" display="off"/>
-</element>
-<element name="S3" library="SparkFun-Electromechanical" package="TACTILE-PTH" value="SWITCH-MOMENTARY-2PTH" x="-81.28" y="-17.78">
-<attribute name="PROD_ID" value=" SWCH-08441" x="-81.28" y="-17.78" size="1.778" layer="27" display="off"/>
-</element>
-<element name="S4" library="SparkFun-Electromechanical" package="TACTILE-PTH" value="SWITCH-MOMENTARY-2PTH" x="-90.17" y="-17.78">
-<attribute name="PROD_ID" value=" SWCH-08441" x="-90.17" y="-17.78" size="1.778" layer="27" display="off"/>
-</element>
-<element name="S5" library="SparkFun-Electromechanical" package="TACTILE-PTH" value="SWITCH-MOMENTARY-2PTH" x="-99.06" y="-17.78">
-<attribute name="PROD_ID" value=" SWCH-08441" x="-99.06" y="-17.78" size="1.778" layer="27" display="off"/>
-</element>
-<element name="S6" library="SparkFun-Electromechanical" package="TACTILE-PTH" value="SWITCH-MOMENTARY-2PTH" x="-107.95" y="-17.78">
-<attribute name="PROD_ID" value=" SWCH-08441" x="-107.95" y="-17.78" size="1.778" layer="27" display="off"/>
-</element>
-<element name="S7" library="SparkFun-Electromechanical" package="TACTILE-PTH" value="SWITCH-MOMENTARY-2PTH" x="-116.84" y="-17.78">
-<attribute name="PROD_ID" value=" SWCH-08441" x="-116.84" y="-17.78" size="1.778" layer="27" display="off"/>
-</element>
 <element name="C1" library="SparkFun-Capacitors" package="CAP-PTH-SMALL" value="0.1uF" x="-119.38" y="-24.13"/>
 </elements>
@@
 <contactref element="U1" pad="13"/>
 <contactref element="R2" pad="P$1"/>
-<contactref element="S1" pad="1"/>
-<wire x1="-36.83" y1="13.97" x2="-66.7512" y2="-15.5194" width="0" layer="19" extent="1-1"/>
 <wire x1="-17.78" y1="2.54" x2="-36.83" y2="13.97" width="0" layer="19" extent="1-1"/>
 </signal>
@@
 <contactref element="U1" pad="14"/>
 <contactref element="R3" pad="P$1"/>
-<contactref element="S2" pad="1"/>
-<wire x1="-24.13" y1="19.05" x2="-75.6412" y2="-15.5194" width="0" layer="19" extent="1-1"/>
-<wire x1="-15.24" y1="2.54" x2="-24.13" y2="19.05" width="0" layer="19" extent="1-1"/>
+<wire x1="-24.13" y1="19.05" x2="-15.24" y2="2.54" width="0" layer="19" extent="1-1"/>
 </signal>
 <signal name="N$3">
 <contactref element="U1" pad="15"/>
 <contactref element="R4" pad="P$1"/>
-<contactref element="S3" pad="1"/>
-<wire x1="-36.83" y1="19.05" x2="-84.5312" y2="-15.5194" width="0" layer="19" extent="1-1"/>
 <wire x1="-15.24" y1="10.16" x2="-36.83" y2="19.05" width="0" layer="19" extent="1-1"/>
 </signal>
@@
 <contactref element="U1" pad="16"/>
 <contactref element="R5" pad="P$1"/>
-<contactref element="S4" pad="1"/>
-<wire x1="-24.13" y1="24.13" x2="-93.4212" y2="-15.5194" width="0" layer="19" extent="1-1"/>
-<wire x1="-17.78" y1="10.16" x2="-24.13" y2="24.13" width="0" layer="19" extent="1-1"/>
+<wire x1="-24.13" y1="24.13" x2="-17.78" y2="10.16" width="0" layer="19" extent="1-1"/>
 </signal>
 <signal name="N$5">
 <contactref element="U1" pad="17"/>
 <contactref element="R7" pad="P$1"/>
-<contactref element="S5" pad="1"/>
-<wire x1="-20.32" y1="10.16" x2="-102.3112" y2="-15.5194" width="0" layer="19" extent="1-1"/>
 <wire x1="-24.13" y1="29.21" x2="-20.32" y2="10.16" width="0" layer="19" extent="1-1"/>
 </signal>
@@
 <contactref element="U1" pad="18"/>
 <contactref element="R8" pad="P$1"/>
-<contactref element="S6" pad="1"/>
-<wire x1="-36.83" y1="29.21" x2="-111.2012" y2="-15.5194" width="0" layer="19" extent="1-1"/>
-<wire x1="-22.86" y1="10.16" x2="-36.83" y2="29.21" width="0" layer="19" extent="1-1"/>
+<wire x1="-36.83" y1="29.21" x2="-22.86" y2="10.16" width="0" layer="19" extent="1-1"/>
 </signal>
 <signal name="N$7">
 <contactref element="U1" pad="19"/>
 <contactref element="R9" pad="P$1"/>
-<contactref element="S7" pad="1"/>
-<wire x1="-25.4" y1="10.16" x2="-120.0912" y2="-15.5194" width="0" layer="19" extent="1-1"/>
 <wire x1="-24.13" y1="34.29" x2="-25.4" y2="10.16" width="0" layer="19" extent="1-1"/>
 </signal>
@@
 <contactref element="T1" pad="E"/>
 <contactref element="D1" pad="K"/>
-<contactref element="S1" pad="3"/>
-<contactref element="S2" pad="3"/>
-<contactref element="S3" pad="3"/>
-<contactref element="S4" pad="3"/>
-<contactref element="S5" pad="3"/>
-<contactref element="S6" pad="3"/>
-<contactref element="S7" pad="3"/>
 <contactref element="U1" pad="8"/>
 <contactref element="U1" pad="22"/>
 <contactref element="C1" pad="2"/>
-<wire x1="-120.0912" y1="-20.0406" x2="-116.84" y2="-24.13" width="0" layer="19" extent="1-1"/>
-<wire x1="-111.2012" y1="-20.0406" x2="-116.84" y2="-24.13" width="0" layer="19" extent="1-1"/>
-<wire x1="-102.3112" y1="-20.0406" x2="-111.2012" y2="-20.0406" width="0" layer="19" extent="1-1"/>
-<wire x1="-93.4212" y1="-20.0406" x2="-102.3112" y2="-20.0406" width="0" layer="19" extent="1-1"/>
-<wire x1="-84.5312" y1="-20.0406" x2="-93.4212" y2="-20.0406" width="0" layer="19" extent="1-1"/>
-<wire x1="-75.6412" y1="-20.0406" x2="-84.5312" y2="-20.0406" width="0" layer="19" extent="1-1"/>
-<wire x1="-66.7512" y1="-20.0406" x2="-75.6412" y2="-20.0406" width="0" layer="19" extent="1-1"/>
-<wire x1="-53.34" y1="-13.97" x2="-66.7512" y2="-20.0406" width="0" layer="19" extent="1-1"/>
+<wire x1="-53.34" y1="-13.97" x2="-116.84" y2="-24.13" width="0" layer="19" extent="1-1"/>
 <wire x1="-57.15" y1="3.81" x2="-53.34" y2="-13.97" width="0" layer="19" extent="1-1"/>
 <wire x1="-33.02" y1="10.16" x2="-57.15" y2="3.81" width="0" layer="19" extent="1-1"/>
@@
 </signal>
 <signal name="GPIO21">
-<contactref element="U1" pad="28"/>
+<contactref element="U1" pad="25"/>
 </signal>
 </signals>
