File: Schematics/MirrorController.sch (EAGLE design)
At the start: 23 parts, among them T1 2N2222, U1 ATMEGA328P_PDIP

Commit message: +I2C Support and temp files removed
Parts:
- removed S1, S2, S3, S4, S5, S6, S7: SWITCH-MOMENTARY-2PTH, SparkFun-Electromechanical:SWITCH-MOMENTARY-2PTH
- R2, R8: value (none) -> 3.9K
- R3, R9: value (none) -> 1K
- R4, R7: value (none) -> 27K
- R5: value (none) -> 10K
Connections:
- net GND: no longer S1.2, S2.2, S3.2, S4.2, S5.2, S6.2, S7.2
- net GPIO21: now also U1.PC2(ADC2); no longer U1.PC5(ADC5/SCL)
- net N$1: no longer S1.1
- net N$2: no longer S2.1
- net N$3: no longer S3.1
- net N$4: no longer S4.1
- net N$5: no longer S5.1
- net N$6: no longer S6.1
- net N$7: no longer S7.1
Other:
- moved on the sheet: R3, R5, R8
